Commit message: Solve orientation problem and added object/cyl

File: hand_simulator/urdf/hand.xacro (robot description, xacro)
@@ -20,7 +20,24 @@
   </xacro:macro>
  <link name="world"/>
+    <link name="table">
+      <visual>
+        <origin rpy="0 0 0" xyz="0 0 0"/>
+        <geometry>
+          <box size="0.5 0.5 0.5" />
+        </geometry>
+        <material name="white"/>
+      </visual>
+      <inertial>
+          <origin xyz="0 0 0.3" rpy="0 0 0"/>
+          <mass value="0.1"/>
+          <inertia
+            ixx="0.0" ixy="0.0" ixz="0.0"
+            iyy="0.0" iyz="0.0"
+            izz="0.0"/>
+        </inertial>
+    </link>
     <link name="base_link">
       <visual>
-          <origin rpy="0. 0 0" xyz="0 0 0"/>
+          <origin rpy="0 0 0" xyz="0 0 0"/>
           <geometry>
             <mesh filename="package://urdf_display/meshes/base_link.STL"/>
@@ -40,5 +57,5 @@
       </inertial>
       <collision>
-        <origin rpy="0.5 0 0" xyz="0 0 0"/>
+        <origin rpy="0 0 0" xyz="0 0 0"/>
         <geometry>
           <mesh filename="package://urdf_display/meshes/base_link.STL"/>
@@ -72,7 +89,213 @@
       </collision>
     </link>
-    <joint name="fixed" type="fixed">
+    <link name="finger_1_2">
+      <visual>
+        <geometry>
+          <mesh filename="package://urdf_display/meshes/proximal_1.STL"/>
+        </geometry>
+        <origin
+          xyz="-0.011 0.007 0.011"
+          rpy="3.1459 0 0"/>
+        <material
+          name="">
+          <xacro:proximal_color/>
+        </material>
+      </visual>
+      <inertial>
+          <origin xyz="0 0 0" rpy="0 0 0"/>
+          <mass value="0.1"/>
+          <inertia
+            ixx="0.0" ixy="0.0" ixz="0.0"
+            iyy="0.0" iyz="0.0"
+            izz="0.0"/>
+      </inertial>
+      <collision>
+        <origin rpy="3.1459 0 0" xyz="-0.011 0.007 0.011"/>
+        <geometry>
+          <mesh filename="package://urdf_display/meshes/proximal_1.STL"/>
+        </geometry>
+      </collision>
+    </link>
+    <link name="finger_1_3">
+      <visual>
+        <geometry>
+          <mesh filename="package://urdf_display/meshes/distal_1.STL"/>
+        </geometry>
+        <origin
+          xyz="-0.077 0.007 0.007"
+          rpy="3.1459 0 0" />
+        <material
+          name="">
+          <xacro:distal_color/>
+        </material>
+      </visual>
+      <inertial>
+          <origin xyz="0 0 0" rpy="0 0 0"/>
+          <mass value="0.1"/>
+          <inertia
+            ixx="0.0" ixy="0.0" ixz="0.0"
+            iyy="0.0" iyz="0.0"
+            izz="0.0"/>
+        </inertial>
+      <collision>
+        <origin rpy="3.1459 0 0" xyz="-0.077 0.007 0.007"/>
+        <geometry>
+          <mesh filename="package://urdf_display/meshes/distal_1.STL"/>
+        </geometry>
+      </collision>
+    </link>
+    <!-- <a> This is strange: Links for Finger 2 but true! </a>-->
+    <link name="finger_2_1">
+      <visual>
+        <geometry>
+          <mesh filename="package://urdf_display/meshes/swivel_1.STL"/>
+        </geometry>
+        <material
+          name="">
+          <xacro:swivel_color/>
+        </material>
+      </visual>
+      <inertial>
+          <origin xyz="0 0 0" rpy="0 0 0"/>
+          <mass value="0.1"/>
+          <inertia
+            ixx="0.0" ixy="0.0" ixz="0.0"
+            iyy="0.0" iyz="0.0"
+            izz="0.0"/>
+        </inertial>
+      <collision>
+        <!-- <origin rpy="0 0 0" xyz="0 0 0"/> -->
+        <geometry>
+          <mesh filename="package://urdf_display/meshes/swivel_1.STL"/>
+        </geometry>
+      </collision>
+    </link>
+    <link name="finger_2_2">
+      <visual>
+        <geometry>
+          <mesh filename="package://urdf_display/meshes/proximal_1.STL"/>
+        </geometry>
+        <origin
+        xyz="-0.011 0.007 0.011"
+        rpy="3.1459 0 0"/>
+        <origin rpy="0 0 0" xyz="0 0 0"/>
+        <material
+          name="">
+          <xacro:proximal_color/>
+        </material>
+      </visual>
+      <inertial>
+          <origin xyz="0 0 0" rpy="0 0 0"/>
+          <mass value="0.1"/>
+          <inertia
+            ixx="0.0" ixy="0.0" ixz="0.0"
+            iyy="0.0" iyz="0.0"
+            izz="0.0"/>
+        </inertial>
+      <collision>
+        <origin rpy="3.1459 0 0" xyz="-0.011 0.007 0.011"/>
+        <geometry>
+          <mesh filename="package://urdf_display/meshes/proximal_1.STL"/>
+        </geometry>
+      </collision>
+    </link>
+    <link name="finger_2_3">
+      <visual>
+        <geometry>
+          <mesh filename="package://urdf_display/meshes/distal_1.STL"/>
+        </geometry>
+        <origin
+        xyz="-0.077 0.007 0.006"
+        rpy="3.1459 0 0" />
+        <origin rpy="0 0 0" xyz="0 0 0"/>
+        <material
+          name="">
+          <xacro:distal_color/>
+        </material>
+      </visual>
+      <inertial>
+          <origin xyz="0 0 0" rpy="0 0 0"/>
+          <mass value="0.1"/>
+          <inertia
+            ixx="0.0" ixy="0.0" ixz="0.0"
+            iyy="0.0" iyz="0.0"
+            izz="0.0"/>
+      </inertial>
+      <collision>
+        <origin rpy="3.1459 0 0" xyz="-0.077 0.007 0.006"/>
+        <geometry>
+          <mesh filename="package://urdf_display/meshes/distal_1.STL"/>
+        </geometry>
+      </collision>
+    </link>
+    <link name="finger_3_2">
+      <visual>
+        <geometry>
+          <mesh filename="package://urdf_display/meshes/proximal_1.STL"/>
+        </geometry>
+        <origin
+        xyz="-0.011 0.007 0.011"
+        rpy="3.1459 0 0"/>
+        <origin rpy="0 0 0" xyz="0 0 0"/>
+        <material
+          name="">
+          <xacro:proximal_color/>
+        </material>
+      </visual>
+      <inertial>
+          <origin xyz="0 0 0" rpy="0 0 0"/>
+          <mass value="0.1"/>
+          <inertia
+            ixx="0.0" ixy="0.0" ixz="0.0"
+            iyy="0.0" iyz="0.0"
+            izz="0.0"/>
+      </inertial>
+      <collision>
+        <origin rpy="3.1459 0 0" xyz="-0.011 0.007 0.011"/>
+        <geometry>
+          <mesh filename="package://urdf_display/meshes/proximal_1.STL"/>
+        </geometry>
+      </collision>
+    </link>
+    <link name="finger_3_3">
+      <visual>
+        <geometry>
+          <mesh filename="package://urdf_display/meshes/distal_1.STL"/>
+        </geometry>
+        <origin
+        xyz="-0.077 0.007 0.006"
+        rpy="3.1459 0 0" />
+        <origin rpy="0 0 0" xyz="0 0 0"/>
+        <material
+          name="">
+          <xacro:distal_color/>
+        </material>
+      </visual>
+      <inertial>
+          <origin xyz="0 0 0" rpy="0 0 0"/>
+          <mass value="0.1"/>
+          <inertia
+            ixx="0.0" ixy="0.0" ixz="0.0"
+            iyy="0.0" iyz="0.0"
+            izz="0.0"/>
+      </inertial>
+      <collision>
+        <origin rpy="3.1459 0 0" xyz="-0.077 0.007 0.006"/>
+        <geometry>
+          <mesh filename="package://urdf_display/meshes/distal_1.STL"/>
+        </geometry>
+      </collision>
+    </link>
+    <joint name="world_to_table" type="fixed">
+      <parent link="world"/>
+      <child link="table"/>
+      <origin xyz="0 0 0.0"/>
+    </joint>
+    <joint name="world_to_base" type="fixed">
       <parent link="world"/>
       <child link="base_link"/>
+      <origin
+        xyz="0.25 0 0.6"
+        rpy="0 1.57 0" />
     </joint>
     <joint name="base_to_finger_1_1" type="revolute">
@@ -85,3 +308,149 @@
         rpy="6.75550818663469E-16 1.97993848419069E-16 -2.77555756156289E-16" />
     </joint>
+    <joint name="finger_1_1_to_finger_1_2" type="revolute">
+      <parent link="finger_1_1"/>
+      <child link="finger_1_2"/>
+      <limit effort="1000.0" lower="-0.1" upper="3.0" velocity="0.5"/>
+      <axis xyz="0 -1 0"/>
+      <origin
+      xyz="0.01 0 0.0186"
+      rpy="-6.20039667432211E-16 0.28 2.22044604925031E-16" />
+    </joint>
+    <joint name="finger_1_2_to_finger_1_3" type="revolute">
+      <parent link="finger_1_2"/>
+      <child link="finger_1_3"/>
+      <limit effort="1000.0" lower="0.0" upper="1.57" velocity="0.5"/>
+      <axis xyz="0 -1 0"/>
+      <origin
+      xyz="0.07600000000000001 0 0.00250000000000002"
+      rpy="0 0 0" />
+    </joint>
+    <joint name="base_to_finger_2_1" type="revolute">
+      <parent link="base_link"/>
+      <child link="finger_2_1"/>
+      <limit effort="1000.0" lower="-2.0" upper="1.57" velocity="0.5"/>
+      <axis xyz="0 0 -1"/>
+      <origin
+      xyz="0.0503973683071413 0.0259999999999999 0.063"
+      rpy="1.22459340959228E-15 -7.33448407631817E-16 -1.66533453693773E-16" />
+      <mimic joint="base_to_finger_1_1" multiplier="-1"/>
+    </joint>
+    <joint name="finger_2_1_to_finger_2_2" type="revolute">
+      <parent link="finger_2_1"/>
+      <child link="finger_2_2"/>
+      <axis xyz="0 -1 0"/>
+      <limit effort="1000.0" lower="-0.1" upper="3.0" velocity="0.5"/>
+      <origin
+      xyz="0.01 0 0.0186"
+      rpy="-1.16908225836102E-15 0.28 1.11022302462515E-16" />
+    </joint>
+    <joint name="finger_2_2_to_finger_2_3" type="revolute">
+      <parent link="finger_2_2"/>
+      <child link="finger_2_3"/>
+      <axis xyz="0 -1 0"/>
+      <limit effort="1000.0" lower="0.0" upper="1.57" velocity="0.5"/>
+      <origin
+      xyz="0.0760000000000001 0 0.00249999999999997"
+      rpy="0 0 0" />
+      <origin xyz="0 2 0"/>
+    </joint>
+    <joint name="base_to_finger_3_2" type="revolute">
+      <parent link="base_link"/>
+      <child link="finger_3_2"/>
+      <axis xyz="0 -1 0"/>
+      <limit effort="1000.0" lower="-0.1" upper="3.0" velocity="0.5"/>
+      <origin
+      xyz="-0.0299999999999996 0 0.0816000000000002"
+      rpy="-5.55111512312578E-17 0.28 3.14159265358979" />
+      <origin xyz="0 0 0.5"/>
+    </joint>
+    <joint name="finger_3_2_to_finger_3_3" type="revolute">
+      <parent link="finger_3_2"/>
+      <child link="finger_3_3"/>
+      <axis xyz="0 -1 0"/>
+      <limit effort="1000.0" lower="0.0" upper="1.57" velocity="0.5"/>
+      <origin
+      xyz="0.0760000000000001 0 0.0025"
+      rpy="-1.48887961834512E-45 -1.0995850059156E-76 -7.38531841236285E-32" />
+      <origin xyz="0 -2 0"/>
+    </joint>
+      <!-- This block connects the head_swivel joint to an actuator (motor), which informs both
+  simulation and visualization of the robot -->
+    <transmission name="finger1_1_trans" type="SimpleTransmission">
+      <type>transmission_interface/SimpleTransmission</type>
+      <actuator name="$finger11_motor">
+          <mechanicalReduction>1</mechanicalReduction>
+      </actuator>
+      <joint name="base_to_finger_1_1">
+          <hardwareInterface>hardware_interface/PositionJointInterface</hardwareInterface>
+      </joint>
+  </transmission>
+  <transmission name="finger1_2_trans" type="SimpleTransmission">
+      <type>transmission_interface/SimpleTransmission</type>
+      <actuator name="$finger12_motor">
+          <mechanicalReduction>1</mechanicalReduction>
+      </actuator>
+      <joint name="finger_1_1_to_finger_1_2">
+          <hardwareInterface>hardware_interface/PositionJointInterface</hardwareInterface>
+      </joint>
+  </transmission>
+  <transmission name="finger1_3_trans" type="SimpleTransmission">
+      <type>transmission_interface/SimpleTransmission</type>
+      <actuator name="$finger13_motor">
+          <mechanicalReduction>1</mechanicalReduction>
+      </actuator>
+      <joint name="finger_1_2_to_finger_1_3">
+          <hardwareInterface>hardware_interface/PositionJointInterface</hardwareInterface>
+      </joint>
+  </transmission>
+  <transmission name="finger2_1_trans" type="SimpleTransmission">
+      <type>transmission_interface/SimpleTransmission</type>
+      <actuator name="$finger21_motor">
+          <mechanicalReduction>1</mechanicalReduction>
+      </actuator>
+      <joint name="base_to_finger_2_1">
+          <hardwareInterface>hardware_interface/PositionJointInterface</hardwareInterface>
+      </joint>
+  </transmission>
+  <transmission name="finger2_2_trans" type="SimpleTransmission">
+      <type>transmission_interface/SimpleTransmission</type>
+      <actuator name="$finger22_motor">
+          <mechanicalReduction>1</mechanicalReduction>
+      </actuator>
+      <joint name="finger_2_1_to_finger_2_2">
+          <hardwareInterface>hardware_interface/PositionJointInterface</hardwareInterface>
+      </joint>
+  </transmission>
+  <transmission name="finger2_3_trans" type="SimpleTransmission">
+      <type>transmission_interface/SimpleTransmission</type>
+      <actuator name="$finger23_motor">
+          <mechanicalReduction>1</mechanicalReduction>
+      </actuator>
+      <joint name="finger_2_2_to_finger_2_3">
+          <hardwareInterface>hardware_interface/PositionJointInterface</hardwareInterface>
+      </joint>
+  </transmission>
+  <transmission name="finger2_3_trans" type="SimpleTransmission">
+      <type>transmission_interface/SimpleTransmission</type>
+      <actuator name="$finger32_motor">
+          <mechanicalReduction>1</mechanicalReduction>
+      </actuator>
+      <joint name="base_to_finger_3_2">
+          <hardwareInterface>hardware_interface/PositionJointInterface</hardwareInterface>
+      </joint>
+  </transmission>
+  <transmission name="finger3_3_trans" type="SimpleTransmission">
+      <type>transmission_interface/SimpleTransmission</type>
+      <actuator name="$finger33_motor">
+          <mechanicalReduction>1</mechanicalReduction>
+      </actuator>
+      <joint name="finger_3_2_to_finger_3_3">
+          <hardwareInterface>hardware_interface/PositionJointInterface</hardwareInterface>
+      </joint>
+  </transmission>
+    <gazebo>
+      <plugin name="gazebo_ros_control" filename="libgazebo_ros_control.so">
+          <robotNamespace>/hand</robotNamespace>
+      </plugin>
+    </gazebo>
 </robot>
