Commit message: Hand object setup

File: hand_simulator/urdf/hand.xacro (robot description, xacro)
@@ -20,26 +20,9 @@
   </xacro:macro>
  <link name="world"/>
-    <link name="table">
-      <visual>
-        <origin rpy="0 0 0" xyz="0 0 0"/>
-        <geometry>
-          <box size="0.5 0.5 0.5" />
-        </geometry>
-        <material name="white"/>
-      </visual>
-      <inertial>
-          <origin xyz="0 0 0.3" rpy="0 0 0"/>
-          <mass value="0.1"/>
-          <inertia
-            ixx="0.0" ixy="0.0" ixz="0.0"
-            iyy="0.0" iyz="0.0"
-            izz="0.0"/>
-        </inertial>
-    </link>
     <link name="base_link">
       <visual>
           <origin rpy="0 0 0" xyz="0 0 0"/>
           <geometry>
-            <mesh filename="package://urdf_display/meshes/base_link.STL"/>
+            <mesh filename="package://hand_simulator/meshes/base_link.STL"/>
           </geometry>
           <material
@@ -59,13 +42,16 @@
         <origin rpy="0 0 0" xyz="0 0 0"/>
         <geometry>
-          <mesh filename="package://urdf_display/meshes/base_link.STL"/>
-        </geometry>
-      </collision>
-    </link>
+          <mesh filename="package://hand_simulator/meshes/base_link.STL"/>
+        </geometry>
+      </collision>
+    </link>
+    <gazebo reference="base_link">
+      <material>Gazebo/Black</material>
+    </gazebo>
   <!-- <a> This is strange: Links for Finger 1 but true! </a>-->
     <link name="finger_1_1">
       <visual>
         <geometry>
-          <mesh filename="package://urdf_display/meshes/swivel_1.STL"/>
+          <mesh filename="package://hand_simulator/meshes/swivel_1.STL"/>
         </geometry>
         <material
@@ -85,12 +71,15 @@
         <!-- <origin rpy="0 0 0" xyz="0 0 0"/> -->
         <geometry>
-          <mesh filename="package://urdf_display/meshes/swivel_1.STL"/>
-        </geometry>
-      </collision>
-    </link>
+          <mesh filename="package://hand_simulator/meshes/swivel_1.STL"/>
+        </geometry>
+      </collision>
+    </link>
+    <gazebo reference="finger_1_1">
+      <material>Gazebo/Red</material>
+    </gazebo>
     <link name="finger_1_2">
       <visual>
         <geometry>
-          <mesh filename="package://urdf_display/meshes/proximal_1.STL"/>
+          <mesh filename="package://hand_simulator/meshes/proximal_1.STL"/>
         </geometry>
         <origin
@@ -113,12 +102,15 @@
         <origin rpy="3.1459 0 0" xyz="-0.011 0.007 0.011"/>
         <geometry>
-          <mesh filename="package://urdf_display/meshes/proximal_1.STL"/>
-        </geometry>
-      </collision>
-    </link>
+          <mesh filename="package://hand_simulator/meshes/proximal_1.STL"/>
+        </geometry>
+      </collision>
+    </link>
+    <gazebo reference="finger_1_2">
+      <material>Gazebo/Red</material>
+    </gazebo>
     <link name="finger_1_3">
       <visual>
         <geometry>
-          <mesh filename="package://urdf_display/meshes/distal_1.STL"/>
+          <mesh filename="package://hand_simulator/meshes/distal_1.STL"/>
         </geometry>
         <origin
@@ -141,13 +133,16 @@
         <origin rpy="3.1459 0 0" xyz="-0.077 0.007 0.007"/>
         <geometry>
-          <mesh filename="package://urdf_display/meshes/distal_1.STL"/>
-        </geometry>
-      </collision>
-    </link>
+          <mesh filename="package://hand_simulator/meshes/distal_1.STL"/>
+        </geometry>
+      </collision>
+    </link>
+    <gazebo reference="finger_1_3">
+      <material>Gazebo/Red</material>
+    </gazebo>
     <!-- <a> This is strange: Links for Finger 2 but true! </a>-->
     <link name="finger_2_1">
       <visual>
         <geometry>
-          <mesh filename="package://urdf_display/meshes/swivel_1.STL"/>
+          <mesh filename="package://hand_simulator/meshes/swivel_1.STL"/>
         </geometry>
         <material
@@ -167,12 +162,15 @@
         <!-- <origin rpy="0 0 0" xyz="0 0 0"/> -->
         <geometry>
-          <mesh filename="package://urdf_display/meshes/swivel_1.STL"/>
-        </geometry>
-      </collision>
-    </link>
+          <mesh filename="package://hand_simulator/meshes/swivel_1.STL"/>
+        </geometry>
+      </collision>
+    </link>
+    <gazebo reference="finger_2_1">
+      <material>Gazebo/Red</material>
+    </gazebo>
     <link name="finger_2_2">
       <visual>
         <geometry>
-          <mesh filename="package://urdf_display/meshes/proximal_1.STL"/>
+          <mesh filename="package://hand_simulator/meshes/proximal_1.STL"/>
         </geometry>
         <origin
@@ -196,12 +194,15 @@
         <origin rpy="3.1459 0 0" xyz="-0.011 0.007 0.011"/>
         <geometry>
-          <mesh filename="package://urdf_display/meshes/proximal_1.STL"/>
-        </geometry>
-      </collision>
-    </link>
+          <mesh filename="package://hand_simulator/meshes/proximal_1.STL"/>
+        </geometry>
+      </collision>
+    </link>
+    <gazebo reference="finger_2_2">
+        <material>Gazebo/Red</material>
+    </gazebo>
     <link name="finger_2_3">
       <visual>
         <geometry>
-          <mesh filename="package://urdf_display/meshes/distal_1.STL"/>
+          <mesh filename="package://hand_simulator/meshes/distal_1.STL"/>
         </geometry>
         <origin
@@ -225,12 +226,15 @@
         <origin rpy="3.1459 0 0" xyz="-0.077 0.007 0.006"/>
         <geometry>
-          <mesh filename="package://urdf_display/meshes/distal_1.STL"/>
-        </geometry>
-      </collision>
-    </link>
+          <mesh filename="package://hand_simulator/meshes/distal_1.STL"/>
+        </geometry>
+      </collision>
+    </link>
+    <gazebo reference="finger_2_3">
+        <material>Gazebo/Red</material>
+    </gazebo>
     <link name="finger_3_2">
       <visual>
         <geometry>
-          <mesh filename="package://urdf_display/meshes/proximal_1.STL"/>
+          <mesh filename="package://hand_simulator/meshes/proximal_1.STL"/>
         </geometry>
         <origin
@@ -254,12 +258,15 @@
         <origin rpy="3.1459 0 0" xyz="-0.011 0.007 0.011"/>
         <geometry>
-          <mesh filename="package://urdf_display/meshes/proximal_1.STL"/>
-        </geometry>
-      </collision>
-    </link>
+          <mesh filename="package://hand_simulator/meshes/proximal_1.STL"/>
+        </geometry>
+      </collision>
+    </link>
+    <gazebo reference="finger_3_2">
+        <material>Gazebo/Red</material>
+    </gazebo>
     <link name="finger_3_3">
       <visual>
         <geometry>
-          <mesh filename="package://urdf_display/meshes/distal_1.STL"/>
+          <mesh filename="package://hand_simulator/meshes/distal_1.STL"/>
         </geometry>
         <origin
@@ -283,19 +290,17 @@
         <origin rpy="3.1459 0 0" xyz="-0.077 0.007 0.006"/>
         <geometry>
-          <mesh filename="package://urdf_display/meshes/distal_1.STL"/>
-        </geometry>
-      </collision>
-    </link>
-    <joint name="world_to_table" type="fixed">
-      <parent link="world"/>
-      <child link="table"/>
-      <origin xyz="0 0 0.0"/>
-    </joint>
+          <mesh filename="package://hand_simulator/meshes/distal_1.STL"/>
+        </geometry>
+      </collision>
+    </link>
+    <gazebo reference="finger_3_3">
+        <material>Gazebo/Red</material>
+    </gazebo>
     <joint name="world_to_base" type="fixed">
       <parent link="world"/>
       <child link="base_link"/>
       <origin
-        xyz="0.25 0 0.6"
-        rpy="0 1.57 0" />
+        xyz="0.37 0 0.5"
+        rpy="0 -1.57 0" />
     </joint>
     <joint name="base_to_finger_1_1" type="revolute">
@@ -392,5 +397,5 @@
       </actuator>
       <joint name="finger_1_1_to_finger_1_2">
-          <hardwareInterface>hardware_interface/PositionJointInterface</hardwareInterface>
+          <hardwareInterface>hardware_interface/EffortJointInterface</hardwareInterface>
       </joint>
   </transmission>
@@ -401,5 +406,5 @@
       </actuator>
       <joint name="finger_1_2_to_finger_1_3">
-          <hardwareInterface>hardware_interface/PositionJointInterface</hardwareInterface>
+          <hardwareInterface>hardware_interface/EffortJointInterface</hardwareInterface>
       </joint>
   </transmission>
@@ -419,5 +424,5 @@
       </actuator>
       <joint name="finger_2_1_to_finger_2_2">
-          <hardwareInterface>hardware_interface/PositionJointInterface</hardwareInterface>
+          <hardwareInterface>hardware_interface/EffortJointInterface</hardwareInterface>
       </joint>
   </transmission>
@@ -428,5 +433,5 @@
       </actuator>
       <joint name="finger_2_2_to_finger_2_3">
-          <hardwareInterface>hardware_interface/PositionJointInterface</hardwareInterface>
+          <hardwareInterface>hardware_interface/EffortJointInterface</hardwareInterface>
       </joint>
   </transmission>
@@ -437,5 +442,5 @@
       </actuator>
       <joint name="base_to_finger_3_2">
-          <hardwareInterface>hardware_interface/PositionJointInterface</hardwareInterface>
+          <hardwareInterface>hardware_interface/EffortJointInterface</hardwareInterface>
       </joint>
   </transmission>
@@ -446,5 +451,5 @@
       </actuator>
       <joint name="finger_3_2_to_finger_3_3">
-          <hardwareInterface>hardware_interface/PositionJointInterface</hardwareInterface>
+          <hardwareInterface>hardware_interface/EffortJointInterface</hardwareInterface>
       </joint>
   </transmission>

File: hand_simulator/urdf/object.urdf (robot description, URDF)
Before this commit: robot cyl, 1 links, 0 joints
Links:
- link cyl_object: geometry collision cylinder length=0.09 radius=0.025; visual cylinder length=0.09 radius=0.025

Commit message: Issues

File: hand_simulator/urdf/hand.xacro (robot description, xacro)
@@ -297,4 +297,5 @@
         <material>Gazebo/Red</material>
     </gazebo>
+    <!-- Joints -->
     <joint name="world_to_base" type="fixed">
       <parent link="world"/>
@@ -321,4 +322,12 @@
       xyz="0.01 0 0.0186"
       rpy="-6.20039667432211E-16 0.28 2.22044604925031E-16" />
+      <axis>
+        <dynamics>
+          <spring_stiffness>1.0</spring_stiffness>
+          <spring_reference>0.0</spring_reference>
+          <damping>0.0</damping>
+          <friction>0.0</friction>
+        </dynamics>
+      </axis>
     </joint>
     <joint name="finger_1_2_to_finger_1_3" type="revolute">

Commit message: Hand control works

File: hand_simulator/urdf/hand.xacro (robot description, xacro)
@@ -308,5 +308,5 @@
       <parent link="base_link"/>
       <child link="finger_1_1"/>
-      <limit effort="1000.0" lower="-2.0" upper="1.57" velocity="0.5"/>
+      <limit effort="1000.0" lower="0." upper="1.57" velocity="0.5"/>
       <axis xyz="0 0 -1"/>
       <origin
@@ -317,17 +317,10 @@
       <parent link="finger_1_1"/>
       <child link="finger_1_2"/>
-      <limit effort="1000.0" lower="-0.1" upper="3.0" velocity="0.5"/>
+      <limit effort="1000.0" lower="-0.1" upper="2.0" velocity="0.5"/>
       <axis xyz="0 -1 0"/>
       <origin
       xyz="0.01 0 0.0186"
       rpy="-6.20039667432211E-16 0.28 2.22044604925031E-16" />
-      <axis>
-        <dynamics>
-          <spring_stiffness>1.0</spring_stiffness>
-          <spring_reference>0.0</spring_reference>
-          <damping>0.0</damping>
-          <friction>0.0</friction>
-        </dynamics>
-      </axis>
+      <dynamics damping="5"/>
     </joint>
     <joint name="finger_1_2_to_finger_1_3" type="revolute">
@@ -339,9 +332,10 @@
       xyz="0.07600000000000001 0 0.00250000000000002"
       rpy="0 0 0" />
+      <dynamics damping="5"/>
     </joint>
     <joint name="base_to_finger_2_1" type="revolute">
       <parent link="base_link"/>
       <child link="finger_2_1"/>
-      <limit effort="1000.0" lower="-2.0" upper="1.57" velocity="0.5"/>
+      <limit effort="1000.0" lower="-1.57" upper="0." velocity="0.5"/>
       <axis xyz="0 0 -1"/>
       <origin
@@ -354,8 +348,9 @@
       <child link="finger_2_2"/>
       <axis xyz="0 -1 0"/>
-      <limit effort="1000.0" lower="-0.1" upper="3.0" velocity="0.5"/>
+      <limit effort="1000.0" lower="-0.1" upper="2.0" velocity="0.5"/>
       <origin
       xyz="0.01 0 0.0186"
       rpy="-1.16908225836102E-15 0.28 1.11022302462515E-16" />
+      <dynamics damping="5"/>
     </joint>
     <joint name="finger_2_2_to_finger_2_3" type="revolute">
@@ -368,4 +363,5 @@
       rpy="0 0 0" />
       <origin xyz="0 2 0"/>
+      <dynamics damping="5"/>
     </joint>
     <joint name="base_to_finger_3_2" type="revolute">
@@ -378,4 +374,5 @@
       rpy="-5.55111512312578E-17 0.28 3.14159265358979" />
       <origin xyz="0 0 0.5"/>
+      <dynamics damping="5"/>
     </joint>
     <joint name="finger_3_2_to_finger_3_3" type="revolute">
@@ -388,4 +385,5 @@
       rpy="-1.48887961834512E-45 -1.0995850059156E-76 -7.38531841236285E-32" />
       <origin xyz="0 -2 0"/>
+      <dynamics damping="5"/>
     </joint>
       <!-- This block connects the head_swivel joint to an actuator (motor), which informs both

Commit message: Grasp confirmed - friction, lift, etc.

File: hand_simulator/urdf/hand.xacro (robot description, xacro)
@@ -19,5 +19,32 @@
     <color rgba="0.106 0.227 0.631 1"/>
   </xacro:macro>
+  <xacro:property name="rubber_friction_coefficient" value="1.16" />
+  <xacro:property name="rubber_contact_stiffness_coefficient" value="1000000.0" />
+  <xacro:property name="rubber_contact_damping_coefficient" value="1.0" />
  <link name="world"/>
+    <link name="rail">
+      <visual>
+          <origin rpy="0 0 0" xyz="0 0 0"/>
+          <geometry>
+            <cylinder length="0.7" radius="0.02"/>
+          </geometry>
+          <material
+            name="">
+            <xacro:base_color/>
+          </material>
+      </visual>
+      <inertial>
+          <origin xyz="0 0 0" rpy="0 0 0"/>
+          <mass value="0.1"/>
+          <inertia
+            ixx="0.0" ixy="0.0" ixz="0.0"
+            iyy="0.0" iyz="0.0"
+            izz="0.0"/>
+      </inertial>
+    </link>
+    <gazebo reference="rail">
+      <selfCollide>true</selfCollide>
+      <material>Gazebo/White</material>
+    </gazebo>
     <link name="base_link">
       <visual>
@@ -47,4 +74,5 @@
     </link>
     <gazebo reference="base_link">
+      <selfCollide>true</selfCollide>
       <material>Gazebo/Black</material>
     </gazebo>
@@ -76,4 +104,5 @@
     </link>
     <gazebo reference="finger_1_1">
+      <selfCollide>true</selfCollide>
       <material>Gazebo/Red</material>
     </gazebo>
@@ -107,4 +136,9 @@
     </link>
     <gazebo reference="finger_1_2">
+      <selfCollide>true</selfCollide>
+      <mu1>${rubber_friction_coefficient}</mu1>
+      <mu2>${rubber_friction_coefficient}</mu2>
+      <kp>${rubber_contact_stiffness_coefficient}</kp>
+      <kd>${rubber_contact_damping_coefficient}</kd>
       <material>Gazebo/Red</material>
     </gazebo>
@@ -138,4 +172,9 @@
     </link>
     <gazebo reference="finger_1_3">
+      <selfCollide>true</selfCollide>
+      <mu1>${rubber_friction_coefficient}</mu1>
+      <mu2>${rubber_friction_coefficient}</mu2>
+      <kp>${rubber_contact_stiffness_coefficient}</kp>
+      <kd>${rubber_contact_damping_coefficient}</kd>
       <material>Gazebo/Red</material>
     </gazebo>
@@ -167,4 +206,5 @@
     </link>
     <gazebo reference="finger_2_1">
+      <selfCollide>true</selfCollide>
       <material>Gazebo/Red</material>
     </gazebo>
@@ -199,4 +239,9 @@
     </link>
     <gazebo reference="finger_2_2">
+        <selfCollide>true</selfCollide>
+        <mu1>${rubber_friction_coefficient}</mu1>
+        <mu2>${rubber_friction_coefficient}</mu2>
+        <kp>${rubber_contact_stiffness_coefficient}</kp>
+        <kd>${rubber_contact_damping_coefficient}</kd>
         <material>Gazebo/Red</material>
     </gazebo>
@@ -231,5 +276,10 @@
     </link>
     <gazebo reference="finger_2_3">
-        <material>Gazebo/Red</material>
+      <selfCollide>true</selfCollide>
+      <mu1>${rubber_friction_coefficient}</mu1>
+      <mu2>${rubber_friction_coefficient}</mu2>
+      <kp>${rubber_contact_stiffness_coefficient}</kp>
+      <kd>${rubber_contact_damping_coefficient}</kd>
+      <material>Gazebo/Red</material>
     </gazebo>
     <link name="finger_3_2">
@@ -263,5 +313,10 @@
     </link>
     <gazebo reference="finger_3_2">
-        <material>Gazebo/Red</material>
+      <selfCollide>true</selfCollide>
+      <mu1>${rubber_friction_coefficient}</mu1>
+      <mu2>${rubber_friction_coefficient}</mu2>
+      <kp>${rubber_contact_stiffness_coefficient}</kp>
+      <kd>${rubber_contact_damping_coefficient}</kd>
+      <material>Gazebo/Red</material>
     </gazebo>
     <link name="finger_3_3">
@@ -295,8 +350,13 @@
     </link>
     <gazebo reference="finger_3_3">
-        <material>Gazebo/Red</material>
+      <selfCollide>true</selfCollide>
+      <mu1>${rubber_friction_coefficient}</mu1>
+      <mu2>${rubber_friction_coefficient}</mu2>
+      <kp>${rubber_contact_stiffness_coefficient}</kp>
+      <kd>${rubber_contact_damping_coefficient}</kd>
+      <material>Gazebo/Red</material>
     </gazebo>
     <!-- Joints -->
-    <joint name="world_to_base" type="fixed">
+    <!-- <joint name="world_to_base" type="fixed">
       <parent link="world"/>
       <child link="base_link"/>
@@ -304,4 +364,21 @@
         xyz="0.37 0 0.5"
         rpy="0 -1.57 0" />
+    </joint> -->
+    <joint name="world_to_rail" type="fixed">
+      <parent link="world"/>
+      <child link="rail"/>
+      <origin
+        xyz="0.37 0 0.35"
+        rpy="0 0 0" />
+    </joint>
+    <joint name="rail_to_base" type="prismatic">
+      <parent link="rail"/>
+      <child link="base_link"/>
+      <axis xyz="1 0 0"/>
+      <limit effort="1000.0" lower="-100." upper="100." velocity="0.5"/>
+      <origin
+        xyz="0.0 0 0.23"
+        rpy="0 -1.57 0" />
+      <dynamics damping="10"/>
     </joint>
     <joint name="base_to_finger_1_1" type="revolute">
@@ -317,5 +394,5 @@
       <parent link="finger_1_1"/>
       <child link="finger_1_2"/>
-      <limit effort="1000.0" lower="-0.1" upper="2.0" velocity="0.5"/>
+      <limit effort="1000.0" lower="-0.1" upper="3.0" velocity="0.5"/>
       <axis xyz="0 -1 0"/>
       <origin
@@ -348,5 +425,5 @@
       <child link="finger_2_2"/>
       <axis xyz="0 -1 0"/>
-      <limit effort="1000.0" lower="-0.1" upper="2.0" velocity="0.5"/>
+      <limit effort="1000.0" lower="-0.1" upper="3.0" velocity="0.5"/>
       <origin
       xyz="0.01 0 0.0186"
@@ -389,5 +466,14 @@
       <!-- This block connects the head_swivel joint to an actuator (motor), which informs both
   simulation and visualization of the robot -->
-    <transmission name="finger1_1_trans" type="SimpleTransmission">
+  <transmission name="lift" type="SimpleTransmission">
+      <type>transmission_interface/SimpleTransmission</type>
+      <actuator name="$lift_motor">
+          <mechanicalReduction>1</mechanicalReduction>
+      </actuator>
+      <joint name="rail_to_base">
+          <hardwareInterface>hardware_interface/PositionJointInterface</hardwareInterface>
+      </joint>
+  </transmission>
+  <transmission name="finger1_1_trans" type="SimpleTransmission">
       <type>transmission_interface/SimpleTransmission</type>
       <actuator name="$finger11_motor">

File: hand_simulator/urdf/object.urdf (robot description, URDF)
Before this commit: robot cyl, 1 links, 0 joints
Links:
- link cyl_object: mass 1.0 -> 0.1
