Commit message: Started with model O

File: hand_simulator/urdf/hand_reflex.xacro (robot description, xacro)
@@ -1,4 +1,4 @@
 <?xml version="1.0"?>
-<robot xmlns:xacro="http://www.ros.org/wiki/xacro" name="hand_model">
+<robot xmlns:xacro="http://www.ros.org/wiki/xacro" name="hand_reflex_model">
  	<xacro:macro name="base_color">
  		<color rgba="0.1 0.1 0.1 1"/>
@@ -27,5 +27,5 @@
           <origin rpy="0 0 0" xyz="0 0 0"/>
           <geometry>
-            <cylinder length="0.7" radius="0.02"/>
+            <cylinder length="0.8" radius="0.02"/>
           </geometry>
           <material

File: hand_simulator/urdf/table.urdf (robot description, URDF)
Before this commit: robot tb, 1 links, 0 joints
Links:
- link table: geometry collision box size=0.5 0.5 0.5
