Commit message: Finished URDF of model O

File: hand_simulator/urdf/hand_O.xacro (robot description, xacro)
@@ -23,79 +23,55 @@
   <xacro:property name="rubber_contact_damping_coefficient" value="1.0" />
   <link name="world"/>
-  <link name="base_link1">
-    <inertial>
-      <origin xyz="0.000000 0.000000 0.025400"/>
-      <mass value="10.0"/>
-      <inertia ixx="1000.0" ixy="0.0" ixz="0.0" iyy="1000.0" iyz="0.0" izz="1000.0"/>
-    </inertial>
-    <!-- <visual>
-      <material name="lightlue">
-        <color rgba="0. 0.3 1.0 1.0"/>
-      </material>
-      <origin rpy="0 1.57079632679 0" xyz="0.000000 0.000000 0.000000"/>
-      <geometry>
-        <box size = "0.098 0.113 0.00762"/>
-      </geometry>
-    </visual> -->
-    <collision>
-      <origin rpy="0 1.57079632679 0" xyz="0.000000 0.000000 0.000000"/>
-      <geometry>
-        <box size = "0.098 0.113 0.00762"/>
-      </geometry>
-    </collision>
-  </link>
-  <gazebo reference="base_link1">
-      <selfCollide>true</selfCollide>
-      <material>Gazebo/Black</material>
-    </gazebo>
-  <link name="base_link2">
-    <inertial>
-      <origin xyz="0.000000 0.000000 0.025400"/>
-      <mass value="10.0"/>
-      <inertia ixx="1000.0" ixy="0.0" ixz="0.0" iyy="1000.0" iyz="0.0" izz="1000.0"/>
-    </inertial>
-    <!-- <visual>
-      <material name="black">
-        <color rgba="0. 0. 0. 1.0"/>
-      </material>
-      <origin rpy="0 1.57079632679 0" xyz="0.000000 0.000000 0.000000"/>
-      <geometry>
-        <box size = "0.098 0.113 0.06"/>
-      </geometry>
-    </visual> -->
-    <collision>
-      <origin rpy="0 1.57079632679 0" xyz="0.000000 0.000000 0.000000"/>
-      <geometry>
-        <box size = "0.098 0.113 0.06"/>
-      </geometry>
-    </collision>
-  </link>
-  <gazebo reference="base_link2">
-      <selfCollide>true</selfCollide>
-      <material>Gazebo/Black</material>
+  <link name="rail">
+      <visual>
+          <origin rpy="0 0 0" xyz="0 0 0"/>
+          <geometry>
+            <cylinder length="0.8" radius="0.02"/>
+          </geometry>
+          <material
+            name="">
+            <xacro:base_color/>
+          </material>
+      </visual>
+      <inertial>
+          <origin xyz="0 0 0" rpy="0 0 0"/>
+          <mass value="0.1"/>
+          <inertia
+            ixx="0.0" ixy="0.0" ixz="0.0"
+            iyy="0.0" iyz="0.0"
+            izz="0.0"/>
+      </inertial>
+    </link>
+    <gazebo reference="rail">
+      <selfCollide>false</selfCollide>
+      <material>Gazebo/White</material>
     </gazebo>
   <link name="base_link">
-    <inertial>
-      <origin xyz="0.000000 0.000000 0.025400"/>
-      <mass value="10.0"/>
-      <inertia ixx="1000.0" ixy="0.0" ixz="0.0" iyy="1000.0" iyz="0.0" izz="1000.0"/>
-    </inertial>
-    <!-- <visual>
-      <material name="lightlue">
-        <color rgba="0. 0.3 1.0 1.0"/>
-      </material>
-      <origin rpy="0 1.57079632679 0" xyz="0.000000 0.000000 0.000000"/>
-      <geometry>
-        <box size = "0.098 0.128 0.003"/>
-      </geometry>
-    </visual> -->
-    <collision>
-      <origin rpy="0 1.57079632679 0" xyz="0.000000 0.000000 0.000000"/>
-      <geometry>
-        <box size = "0.098 0.128 0.003"/>
-      </geometry>
-    </collision>
-  </link>
-  <gazebo reference="base_link">
+      <visual>
+          <origin rpy="1.57 0 -1.57" xyz="0.06 0.017 0"/>
+          <geometry>
+            <mesh filename="package://hand_simulator/meshes/base_link.STL"/>
+          </geometry>
+          <material
+            name="">
+            <xacro:base_color/>
+          </material>
+      </visual>
+      <inertial>
+          <origin xyz="0 0 0" rpy="0 0 0"/>
+          <mass value="0.1"/>
+          <inertia
+            ixx="0.0" ixy="0.0" ixz="0.0"
+            iyy="0.0" iyz="0.0"
+            izz="0.0"/>
+      </inertial>
+      <!-- <collision>
+        <origin rpy="1.57 0 -1.57" xyz="0.06 0.017 0"/>
+        <geometry>
+          <mesh filename="package://hand_simulator/meshes/base_link.STL"/>
+        </geometry>
+      </collision> -->
+    </link>
+    <gazebo reference="base_link">
       <selfCollide>true</selfCollide>
       <material>Gazebo/Black</material>
@@ -120,10 +96,10 @@
       </geometry>
     </visual>
-    <collision>
+    <!-- <collision>
       <origin rpy="0 1.57 0 " xyz="0.00 0.0 0.00" />
       <geometry>
         <cylinder length="0.002" radius="0.018" />
       </geometry>
-    </collision>
+    </collision> -->
   </link>
   <gazebo reference="finger_1_1">
@@ -150,15 +126,106 @@
     </visual>
     <collision>
-      <origin rpy="1.5707 0 0" xyz="0.00 0.032 0.00" />
-      <geometry>
-        <box size="0.02400 0.018 0.08340" />
+      <origin rpy="0 -3.141592 2.4" xyz="-0.00 0.0753 0.008" />
+      <geometry>
+        <mesh filename="package://openhand_simulator/meshes/proximal_O.STL" scale="0.00100 0.00100 0.00100" />
       </geometry>
     </collision>
   </link>
   <gazebo reference="finger_1_2">
-      <selfCollide>true</selfCollide>
+      <selfCollide>ture</selfCollide>
       <material>Gazebo/Red</material>
     </gazebo>
   <link name="finger_1_3">
+    <inertial>
+          <origin xyz="0 0 0" rpy="0 0 0"/>
+          <mass value="0.1"/>
+          <inertia
+            ixx="0.0" ixy="0.0" ixz="0.0"
+            iyy="0.0" iyz="0.0"
+            izz="0.0"/>
+    </inertial>
+    <visual>
+      <material name="white">
+        <color rgba="1.0 1.0 1.0 1.0" />
+      </material>
+      <origin rpy="0 0 -2.4962" xyz="-0.0179 0.0459 -0.008" />
+      <geometry>
+        <mesh filename="package://openhand_simulator/meshes/distal_O.STL" scale="0.00100 0.00100 0.00100" />
+      </geometry>
+    </visual>
+    <collision>
+      <origin rpy="0 0 -2.4962" xyz="-0.0179 0.0459 -0.008" />
+      <geometry>
+        <mesh filename="package://openhand_simulator/meshes/distal_O.STL" scale="0.00100 0.00100 0.00100" />
+      </geometry>
+    </collision>
+  </link>
+  <gazebo reference="finger_1_3">
+      <selfCollide>true</selfCollide>
+      <mu1>${rubber_friction_coefficient}</mu1>
+      <mu2>${rubber_friction_coefficient}</mu2>
+      <kp>${rubber_contact_stiffness_coefficient}</kp>
+      <kd>${rubber_contact_damping_coefficient}</kd>
+      <material>Gazebo/Red</material>
+    </gazebo>
+  <link name="finger_2_1">
+    <inertial>
+          <origin xyz="0 0 0" rpy="0 0 0"/>
+          <mass value="0.1"/>
+          <inertia
+            ixx="0.0" ixy="0.0" ixz="0.0"
+            iyy="0.0" iyz="0.0"
+            izz="0.0"/>
+      </inertial>
+    <visual>
+      <material name="white">
+        <color rgba="1.0 1.0 1.0 1.0" />
+      </material>
+      <origin rpy="1.57 3.14159 -1.57" xyz="-0.00 0.0 0.00" />
+      <geometry>
+        <mesh filename="package://hand_simulator/meshes/swivel_1.STL"/>
+      </geometry>
+    </visual>
+    <!-- <collision>
+      <origin rpy="0 1.57 0 " xyz="0.00 0.0 0.00" />
+      <geometry>
+        <cylinder length="0.002" radius="0.018" />
+      </geometry>
+    </collision> -->
+  </link>
+  <gazebo reference="finger_2_1">
+      <selfCollide>true</selfCollide>
+      <material>Gazebo/Red</material>
+    </gazebo>
+  <link name="finger_2_2">
+    <inertial>
+          <origin xyz="0 0 0" rpy="0 0 0"/>
+          <mass value="0.1"/>
+          <inertia
+            ixx="0.0" ixy="0.0" ixz="0.0"
+            iyy="0.0" iyz="0.0"
+            izz="0.0"/>
+      </inertial>
+    <visual>
+      <material name="white">
+        <color rgba="1.0 1.0 1.0 1.0" />
+      </material>
+      <origin rpy="0 -3.141592 2.4" xyz="-0.00 0.0753 0.008" />
+      <geometry>
+        <mesh filename="package://openhand_simulator/meshes/proximal_O.STL" scale="0.00100 0.00100 0.00100" />
+      </geometry>
+    </visual>
+    <collision>
+      <origin rpy="0 -3.141592 2.4" xyz="-0.00 0.0753 0.008" />
+      <geometry>
+        <mesh filename="package://openhand_simulator/meshes/proximal_O.STL" scale="0.00100 0.00100 0.00100" />
+      </geometry>
+    </collision>
+  </link>
+  <gazebo reference="finger_2_2">
+      <selfCollide>true</selfCollide>
+      <material>Gazebo/Red</material>
+    </gazebo>
+  <link name="finger_2_3">
     <inertial>
       <origin xyz="-0.015875 -0.009000 -0.071550" />
@@ -182,68 +249,42 @@
     </collision>
   </link>
-  <gazebo reference="finger_1_3">
-      <selfCollide>true</selfCollide>
-      <material>Gazebo/Red</material>
-    </gazebo>
-  <link name="finger_2_1">
-    <inertial>
-          <origin xyz="0 0 0" rpy="0 0 0"/>
-          <mass value="0.1"/>
-          <inertia
-            ixx="0.0" ixy="0.0" ixz="0.0"
-            iyy="0.0" iyz="0.0"
-            izz="0.0"/>
-      </inertial>
-    <visual>
-      <material name="white">
-        <color rgba="1.0 1.0 1.0 1.0" />
-      </material>
-      <origin rpy="1.57 3.14159 -1.57" xyz="-0.00 0.0 0.00" />
-      <geometry>
-        <!-- <cylinder length="0.002" radius="0.018" /> -->
-        <mesh filename="package://hand_simulator/meshes/swivel_1.STL"/>
-      </geometry>
-    </visual>
-    <collision>
-      <origin rpy="0 1.57 0 " xyz="0.00 0.0 0.00" />
-      <geometry>
-        <cylinder length="0.002" radius="0.018" />
-      </geometry>
-    </collision>
-  </link>
-  <gazebo reference="finger_2_1">
-      <selfCollide>true</selfCollide>
-      <material>Gazebo/Red</material>
-    </gazebo>
-  <link name="finger_2_2">
-    <inertial>
-          <origin xyz="0 0 0" rpy="0 0 0"/>
-          <mass value="0.1"/>
-          <inertia
-            ixx="0.0" ixy="0.0" ixz="0.0"
-            iyy="0.0" iyz="0.0"
-            izz="0.0"/>
-      </inertial>
-    <visual>
-      <material name="white">
-        <color rgba="1.0 1.0 1.0 1.0" />
-      </material>
-      <origin rpy="0 -3.141592 2.4" xyz="-0.00 0.0753 0.008" />
-      <geometry>
-        <mesh filename="package://openhand_simulator/meshes/proximal_O.STL" scale="0.00100 0.00100 0.00100" />
-      </geometry>
-    </visual>
-    <collision>
-      <origin rpy="1.5707 0 0" xyz="0.00 0.032 0.00" />
-      <geometry>
-        <box size="0.02400 0.018 0.08340" />
-      </geometry>
-    </collision>
-  </link>
-  <gazebo reference="finger_2_2">
-      <selfCollide>true</selfCollide>
-      <material>Gazebo/Red</material>
-    </gazebo>
-  <link name="finger_2_3">
+  <gazebo reference="finger_2_3">
+      <selfCollide>true</selfCollide>
+      <mu1>${rubber_friction_coefficient}</mu1>
+      <mu2>${rubber_friction_coefficient}</mu2>
+      <kp>${rubber_contact_stiffness_coefficient}</kp>
+      <kd>${rubber_contact_damping_coefficient}</kd>
+      <material>Gazebo/Red</material>
+    </gazebo>
+  <link name="finger_3_2">
+    <inertial>
+          <origin xyz="0 0 0" rpy="0 0 0"/>
+          <mass value="0.1"/>
+          <inertia
+            ixx="0.0" ixy="0.0" ixz="0.0"
+            iyy="0.0" iyz="0.0"
+            izz="0.0"/>
+    </inertial>
+    <visual>
+      <material name="white">
+        <color rgba="1.0 1.0 1.0 1.0" />
+      </material>
+      <origin rpy="0 -3.141592 2.4" xyz="-0.00 0.0753 0.008" />
+      <geometry>
+        <mesh filename="package://openhand_simulator/meshes/proximal_O.STL" scale="0.00100 0.00100 0.00100" />
+      </geometry>
+    </visual>
+    <collision>
+      <origin rpy="0 -3.141592 2.4" xyz="-0.00 0.0753 0.008" />
+      <geometry>
+        <mesh filename="package://openhand_simulator/meshes/proximal_O.STL" scale="0.00100 0.00100 0.00100" />
+      </geometry>
+    </collision>
+  </link>
+  <gazebo reference="finger_3_2">
+      <selfCollide>false</selfCollide>
+      <material>Gazebo/Red</material>
+    </gazebo>
+  <link name="finger_3_3">
     <inertial>
       <origin xyz="-0.015875 -0.009000 -0.071550" />
@@ -267,76 +308,35 @@
     </collision>
   </link>
-  <gazebo reference="finger_2_3">
-      <selfCollide>true</selfCollide>
-      <material>Gazebo/Red</material>
-    </gazebo>
-<!--
-  <link name="finger_3_2">
-    <inertial>
-      <origin xyz="-0.015875 -0.009000 -0.071550" />
-      <mass value="1.0" />
-      <inertia ixx="1.0" ixy="0.0" ixz="0.0" iyy="1.0" iyz="0.0" izz="1.0" />
-    </inertial>
-    <visual>
-      <material name="white">
-        <color rgba="1.0 1.0 1.0 1.0" />
-      </material>
-      <origin rpy="0 -3.141592 2.4" xyz="-0.00 0.0753 0.008" />
-      <geometry>
-        <mesh filename="package://openhand_simulator/meshes/proximal_O.STL" scale="0.00100 0.00100 0.00100" />
-      </geometry>
-    </visual>
-    <collision>
-      <origin rpy="1.5707 0 0" xyz="0.00 0.032 0.00" />
-      <geometry>
-        <box size="0.02400 0.018 0.08340" />
-      </geometry>
-    </collision>
-  </link>
-  <link name="finger_3_3">
-    <inertial>
-      <origin xyz="-0.015875 -0.009000 -0.071550" />
-      <mass value="1.0" />
-      <inertia ixx="1.0" ixy="0.0" ixz="0.0" iyy="1.0" iyz="0.0" izz="1.0" />
-    </inertial>
-    <visual>
-      <material name="white">
-        <color rgba="1.0 1.0 1.0 1.0" />
-      </material>
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
File: hand_simulator/urdf/hand_reflex.xacro (robot description, xacro)
@@ -314,4 +314,37 @@
     <gazebo reference="finger_3_2">
       <selfCollide>true</selfCollide>
+      <material>Gazebo/Red</material>
+    </gazebo>
+    <link name="finger_3_3">
+      <visual>
+        <geometry>
+          <mesh filename="package://hand_simulator/meshes/distal_1.STL"/>
+        </geometry>
+        <origin
+        xyz="-0.077 0.007 0.006"
+        rpy="3.1459 0 0" />
+        <origin rpy="0 0 0" xyz="0 0 0"/>
+        <material
+          name="">
+          <xacro:distal_color/>
+        </material>
+      </visual>
+      <inertial>
+          <origin xyz="0 0 0" rpy="0 0 0"/>
+          <mass value="0.1"/>
+          <inertia
+            ixx="0.0" ixy="0.0" ixz="0.0"
+            iyy="0.0" iyz="0.0"
+            izz="0.0"/>
+      </inertial>
+      <collision>
+        <origin rpy="3.1459 0 0" xyz="-0.077 0.007 0.006"/>
+        <geometry>
+          <mesh filename="package://hand_simulator/meshes/distal_1.STL"/>
+        </geometry>
+      </collision>
+    </link>
+    <gazebo reference="finger_3_3">
+      <selfCollide>true</selfCollide>
       <mu1>${rubber_friction_coefficient}</mu1>
       <mu2>${rubber_friction_coefficient}</mu2>
@@ -320,49 +353,5 @@
       <material>Gazebo/Red</material>
     </gazebo>
-    <link name="finger_3_3">
-      <visual>
-        <geometry>
-          <mesh filename="package://hand_simulator/meshes/distal_1.STL"/>
-        </geometry>
-        <origin
-        xyz="-0.077 0.007 0.006"
-        rpy="3.1459 0 0" />
-        <origin rpy="0 0 0" xyz="0 0 0"/>
-        <material
-          name="">
-          <xacro:distal_color/>
-        </material>
-      </visual>
-      <inertial>
-          <origin xyz="0 0 0" rpy="0 0 0"/>
-          <mass value="0.1"/>
-          <inertia
-            ixx="0.0" ixy="0.0" ixz="0.0"
-            iyy="0.0" iyz="0.0"
-            izz="0.0"/>
-      </inertial>
-      <collision>
-        <origin rpy="3.1459 0 0" xyz="-0.077 0.007 0.006"/>
-        <geometry>
-          <mesh filename="package://hand_simulator/meshes/distal_1.STL"/>
-        </geometry>
-      </collision>
-    </link>
-    <gazebo reference="finger_3_3">
-      <selfCollide>true</selfCollide>
-      <mu1>${rubber_friction_coefficient}</mu1>
-      <mu2>${rubber_friction_coefficient}</mu2>
-      <kp>${rubber_contact_stiffness_coefficient}</kp>
-      <kd>${rubber_contact_damping_coefficient}</kd>
-      <material>Gazebo/Red</material>
-    </gazebo>
     <!-- Joints -->
-    <!-- <joint name="world_to_base" type="fixed">
-      <parent link="world"/>
-      <child link="base_link"/>
-      <origin
-        xyz="0.37 0 0.5"
-        rpy="0 -1.57 0" />
-    </joint> -->
     <joint name="world_to_rail" type="fixed">
       <parent link="world"/>

File: hand_simulator/urdf/table.urdf (robot description, URDF)
Before this commit: robot tb, 1 links, 0 joints
Links:
- link table: geometry collision box size=0.5 0.5 0.5; visual box size=0.5 0.5 0.5

Commit message: Setup of Model T42

File: hand_simulator/urdf/hand_O.xacro (robot description, xacro)
@@ -283,5 +283,5 @@
   </link>
   <gazebo reference="finger_3_2">
-      <selfCollide>false</selfCollide>
+      <selfCollide>true</selfCollide>
       <material>Gazebo/Red</material>
     </gazebo>
@@ -327,8 +327,10 @@
     <parent link="rail"/>
     <child link="base_link"/>
-    <limit effort="1000.0" lower="-100." upper="100." velocity="0.5"/>
+    <axis xyz="0 1 0"/>
+    <limit effort="1000.0" lower="-100." upper="100." velocity="10"/>
     <origin
-      xyz="-0.06 0 0.23"
+      xyz="-0.06 0 -0.19"
       rpy="-1.57 0 0" />
+    <dynamics damping="10"/>
   </joint>
  <joint name="base_to_finger_1_1" type="revolute">
@@ -336,5 +338,5 @@
    <parent link="base_link" />
    <child link="finger_1_1" />
-   <limit effort="1000" lower="0" upper="1.57" velocity="0.5" />
+   <limit effort="1000" lower="0" upper="1.57" velocity="100" />
    <axis xyz="1 0 0" />
    <dynamics damping="5" friction="0.0" />
@@ -344,5 +346,5 @@
    <parent link="finger_1_1" />
    <child link="finger_1_2" />
-   <limit effort="1000.0" lower="-0.1" upper="3.0" velocity="0.5"/>
+   <limit effort="1000.0" lower="-0.1" upper="3.0" velocity="10"/>
    <axis xyz="0 0 1" />
    <dynamics damping="5" friction="0.0" />
@@ -352,5 +354,5 @@
    <parent link="finger_1_2" />
    <child link="finger_1_3" />
-   <limit effort="1000.0" lower="0.0" upper="1.57" velocity="0.5"/>
+   <limit effort="1000.0" lower="0.0" upper="1.27" velocity="10"/>
    <axis xyz="0 0 1" />
    <dynamics damping="5" friction="0.0" />
@@ -360,5 +362,5 @@
     <parent link="base_link" />
     <child link="finger_2_1" />
-    <limit effort="1000" lower="-1.57" upper="0" velocity="200" />
+    <limit effort="1000" lower="-1.57" upper="0" velocity="100" />
     <axis xyz="1 0 0" />
     <dynamics damping="5" friction="0.0" />
@@ -368,5 +370,5 @@
     <parent link="finger_2_1" />
     <child link="finger_2_2" />
-    <limit effort="10000" lower="-0.1" upper="3.0" velocity="200" />
+    <limit effort="1000" lower="-0.1" upper="3.0" velocity="10" />
     <axis xyz="0 0 1" />
     <dynamics damping="5" friction="0.0" />
@@ -376,5 +378,5 @@
     <parent link="finger_2_2" />
     <child link="finger_2_3" />
-    <limit effort="10000" lower="0.0" upper="1.57" velocity="200" />
+    <limit effort="1000" lower="0.0" upper="1.27" velocity="10" />
     <axis xyz="0 0 1" />
     <dynamics damping="5" friction="0.0" />
@@ -384,5 +386,5 @@
     <parent link="base_link" />
     <child link="finger_3_2" />
-    <limit effort="1000" lower="-0.1" upper="3.0" velocity="200" />
+    <limit effort="1000" lower="-0.1" upper="3.0" velocity="10" />
     <axis xyz="0 0 1" />
     <dynamics damping="5" friction="0.0" />
@@ -392,5 +394,5 @@
     <parent link="finger_3_2" />
     <child link="finger_3_3" />
-    <limit effort="10000" lower="0.0" upper="1.57" velocity="200" />
+    <limit effort="1000" lower="0.0" upper="1.27" velocity="10" />
     <axis xyz="0 0 1" />
     <dynamics damping="5" friction="0.0" />
@@ -422,4 +424,5 @@
       <joint name="finger_1_1_to_finger_1_2">
           <hardwareInterface>hardware_interface/EffortJointInterface</hardwareInterface>
+          <!-- <hardwareInterface>hardware_interface/PositionJointInterface</hardwareInterface> -->
       </joint>
   </transmission>
@@ -431,4 +434,5 @@
       <joint name="finger_1_2_to_finger_1_3">
           <hardwareInterface>hardware_interface/EffortJointInterface</hardwareInterface>
+          <!-- <hardwareInterface>hardware_interface/PositionJointInterface</hardwareInterface> -->
       </joint>
   </transmission>
@@ -449,4 +453,5 @@
       <joint name="finger_2_1_to_finger_2_2">
           <hardwareInterface>hardware_interface/EffortJointInterface</hardwareInterface>
+          <!-- <hardwareInterface>hardware_interface/PositionJointInterface</hardwareInterface> -->
       </joint>
   </transmission>
@@ -458,4 +463,5 @@
       <joint name="finger_2_2_to_finger_2_3">
           <hardwareInterface>hardware_interface/EffortJointInterface</hardwareInterface>
+          <!-- <hardwareInterface>hardware_interface/PositionJointInterface</hardwareInterface> -->
       </joint>
   </transmission>
@@ -467,4 +473,5 @@
       <joint name="base_to_finger_3_2">
           <hardwareInterface>hardware_interface/EffortJointInterface</hardwareInterface>
+          <!-- <hardwareInterface>hardware_interface/PositionJointInterface</hardwareInterface> -->
       </joint>
   </transmission>
@@ -476,4 +483,5 @@
       <joint name="finger_3_2_to_finger_3_3">
           <hardwareInterface>hardware_interface/EffortJointInterface</hardwareInterface>
+          <!-- <hardwareInterface>hardware_interface/PositionJointInterface</hardwareInterface> -->
       </joint>
   </transmission>

Commit message: Correction - model_O

File: hand_simulator/urdf/hand_O.xacro (robot description, xacro)
@@ -328,7 +328,7 @@
     <child link="base_link"/>
     <axis xyz="0 1 0"/>
-    <limit effort="1000.0" lower="-100." upper="100." velocity="10"/>
+    <limit effort="1000.0" lower="-100." upper="100." velocity="4"/>
     <origin
-      xyz="-0.06 0 -0.19"
+      xyz="-0.06 0 0.42"
       rpy="-1.57 0 0" />
     <dynamics damping="10"/>
