Commit message: T42 urdf

File: hand_simulator/urdf/hand_O.xacro (robot description, xacro)
@@ -49,5 +49,5 @@
   <link name="base_link">
       <visual>
-          <origin rpy="1.57 0 -1.57" xyz="0.06 0.017 0"/>
+          <origin rpy="1.57 0 -1.57" xyz="0 0 0"/>
           <geometry>
             <mesh filename="package://hand_simulator/meshes/base_link.STL"/>
@@ -122,11 +122,11 @@
       <origin rpy="0 -3.141592 2.4" xyz="-0.00 0.0753 0.008" />
       <geometry>
-        <mesh filename="package://openhand_simulator/meshes/proximal_O.STL" scale="0.00100 0.00100 0.00100" />
-      </geometry>
-    </visual>
-    <collision>
-      <origin rpy="0 -3.141592 2.4" xyz="-0.00 0.0753 0.008" />
-      <geometry>
-        <mesh filename="package://openhand_simulator/meshes/proximal_O.STL" scale="0.00100 0.00100 0.00100" />
+        <mesh filename="package://hand_simulator/meshes/proximal_O.STL" scale="0.00100 0.00100 0.00100" />
+      </geometry>
+    </visual>
+    <collision>
+      <origin rpy="0 -3.141592 2.4" xyz="-0.00 0.0753 0.008" />
+      <geometry>
+        <mesh filename="package://hand_simulator/meshes/proximal_O.STL" scale="0.00100 0.00100 0.00100" />
       </geometry>
     </collision>
@@ -151,11 +151,11 @@
       <origin rpy="0 0 -2.4962" xyz="-0.0179 0.0459 -0.008" />
       <geometry>
-        <mesh filename="package://openhand_simulator/meshes/distal_O.STL" scale="0.00100 0.00100 0.00100" />
-      </geometry>
-    </visual>
-    <collision>
-      <origin rpy="0 0 -2.4962" xyz="-0.0179 0.0459 -0.008" />
-      <geometry>
-        <mesh filename="package://openhand_simulator/meshes/distal_O.STL" scale="0.00100 0.00100 0.00100" />
+        <mesh filename="package://hand_simulator/meshes/distal_O.STL" scale="0.00100 0.00100 0.00100" />
+      </geometry>
+    </visual>
+    <collision>
+      <origin rpy="0 0 -2.4962" xyz="-0.0179 0.0459 -0.008" />
+      <geometry>
+        <mesh filename="package://hand_simulator/meshes/distal_O.STL" scale="0.00100 0.00100 0.00100" />
       </geometry>
     </collision>
@@ -213,11 +213,11 @@
       <origin rpy="0 -3.141592 2.4" xyz="-0.00 0.0753 0.008" />
       <geometry>
-        <mesh filename="package://openhand_simulator/meshes/proximal_O.STL" scale="0.00100 0.00100 0.00100" />
-      </geometry>
-    </visual>
-    <collision>
-      <origin rpy="0 -3.141592 2.4" xyz="-0.00 0.0753 0.008" />
-      <geometry>
-        <mesh filename="package://openhand_simulator/meshes/proximal_O.STL" scale="0.00100 0.00100 0.00100" />
+        <mesh filename="package://hand_simulator/meshes/proximal_O.STL" scale="0.00100 0.00100 0.00100" />
+      </geometry>
+    </visual>
+    <collision>
+      <origin rpy="0 -3.141592 2.4" xyz="-0.00 0.0753 0.008" />
+      <geometry>
+        <mesh filename="package://hand_simulator/meshes/proximal_O.STL" scale="0.00100 0.00100 0.00100" />
       </geometry>
     </collision>
@@ -239,11 +239,11 @@
       <origin rpy="0 0 -2.4962" xyz="-0.0179 0.0459 -0.008" />
       <geometry>
-        <mesh filename="package://openhand_simulator/meshes/distal_O.STL" scale="0.00100 0.00100 0.00100" />
-      </geometry>
-    </visual>
-    <collision>
-      <origin rpy="0 0 -2.4962" xyz="-0.0179 0.0459 -0.008" />
-      <geometry>
-        <mesh filename="package://openhand_simulator/meshes/distal_O.STL" scale="0.00100 0.00100 0.00100" />
+        <mesh filename="package://hand_simulator/meshes/distal_O.STL" scale="0.00100 0.00100 0.00100" />
+      </geometry>
+    </visual>
+    <collision>
+      <origin rpy="0 0 -2.4962" xyz="-0.0179 0.0459 -0.008" />
+      <geometry>
+        <mesh filename="package://hand_simulator/meshes/distal_O.STL" scale="0.00100 0.00100 0.00100" />
       </geometry>
     </collision>
@@ -272,11 +272,11 @@
       <origin rpy="0 -3.141592 2.4" xyz="-0.00 0.0753 0.008" />
       <geometry>
-        <mesh filename="package://openhand_simulator/meshes/proximal_O.STL" scale="0.00100 0.00100 0.00100" />
-      </geometry>
-    </visual>
-    <collision>
-      <origin rpy="0 -3.141592 2.4" xyz="-0.00 0.0753 0.008" />
-      <geometry>
-        <mesh filename="package://openhand_simulator/meshes/proximal_O.STL" scale="0.00100 0.00100 0.00100" />
+        <mesh filename="package://hand_simulator/meshes/proximal_O.STL" scale="0.00100 0.00100 0.00100" />
+      </geometry>
+    </visual>
+    <collision>
+      <origin rpy="0 -3.141592 2.4" xyz="-0.00 0.0753 0.008" />
+      <geometry>
+        <mesh filename="package://hand_simulator/meshes/proximal_O.STL" scale="0.00100 0.00100 0.00100" />
       </geometry>
     </collision>
@@ -298,11 +298,11 @@
       <origin rpy="0 0 -2.4962" xyz="-0.0179 0.0459 -0.008" />
       <geometry>
-        <mesh filename="package://openhand_simulator/meshes/distal_O.STL" scale="0.00100 0.00100 0.00100" />
-      </geometry>
-    </visual>
-    <collision>
-      <origin rpy="0 0 -2.4962" xyz="-0.0179 0.0459 -0.008" />
-      <geometry>
-        <mesh filename="package://openhand_simulator/meshes/distal_O.STL" scale="0.00100 0.00100 0.00100" />
+        <mesh filename="package://hand_simulator/meshes/distal_O.STL" scale="0.00100 0.00100 0.00100" />
+      </geometry>
+    </visual>
+    <collision>
+      <origin rpy="0 0 -2.4962" xyz="-0.0179 0.0459 -0.008" />
+      <geometry>
+        <mesh filename="package://hand_simulator/meshes/distal_O.STL" scale="0.00100 0.00100 0.00100" />
       </geometry>
     </collision>

Commit message: Tuned URDF's

File: hand_simulator/urdf/hand_O.xacro (robot description, xacro)
@@ -49,5 +49,5 @@
   <link name="base_link">
       <visual>
-          <origin rpy="1.57 0 -1.57" xyz="0 0 0"/>
+          <origin rpy="1.57 0 -1.57" xyz="0.06 0.017 0"/>
           <geometry>
             <mesh filename="package://hand_simulator/meshes/base_link.STL"/>
@@ -133,5 +133,5 @@
   </link>
   <gazebo reference="finger_1_2">
-      <selfCollide>ture</selfCollide>
+      <selfCollide>true</selfCollide>
       <material>Gazebo/Red</material>
     </gazebo>
@@ -338,5 +338,5 @@
    <parent link="base_link" />
    <child link="finger_1_1" />
-   <limit effort="1000" lower="0" upper="1.57" velocity="100" />
+   <limit effort="1000" lower="0" upper="1.57" velocity="200" />
    <axis xyz="1 0 0" />
    <dynamics damping="5" friction="0.0" />
@@ -362,5 +362,5 @@
     <parent link="base_link" />
     <child link="finger_2_1" />
-    <limit effort="1000" lower="-1.57" upper="0" velocity="100" />
+    <limit effort="1000" lower="-1.57" upper="0" velocity="200" />
     <axis xyz="1 0 0" />
     <dynamics damping="5" friction="0.0" />
@@ -424,5 +424,4 @@
       <joint name="finger_1_1_to_finger_1_2">
           <hardwareInterface>hardware_interface/EffortJointInterface</hardwareInterface>
-          <!-- <hardwareInterface>hardware_interface/PositionJointInterface</hardwareInterface> -->
       </joint>
   </transmission>
@@ -434,5 +433,4 @@
       <joint name="finger_1_2_to_finger_1_3">
           <hardwareInterface>hardware_interface/EffortJointInterface</hardwareInterface>
-          <!-- <hardwareInterface>hardware_interface/PositionJointInterface</hardwareInterface> -->
       </joint>
   </transmission>
@@ -453,5 +451,4 @@
       <joint name="finger_2_1_to_finger_2_2">
           <hardwareInterface>hardware_interface/EffortJointInterface</hardwareInterface>
-          <!-- <hardwareInterface>hardware_interface/PositionJointInterface</hardwareInterface> -->
       </joint>
   </transmission>
@@ -463,5 +460,4 @@
       <joint name="finger_2_2_to_finger_2_3">
           <hardwareInterface>hardware_interface/EffortJointInterface</hardwareInterface>
-          <!-- <hardwareInterface>hardware_interface/PositionJointInterface</hardwareInterface> -->
       </joint>
   </transmission>
@@ -473,5 +469,4 @@
       <joint name="base_to_finger_3_2">
           <hardwareInterface>hardware_interface/EffortJointInterface</hardwareInterface>
-          <!-- <hardwareInterface>hardware_interface/PositionJointInterface</hardwareInterface> -->
       </joint>
   </transmission>
@@ -483,5 +478,4 @@
       <joint name="finger_3_2_to_finger_3_3">
           <hardwareInterface>hardware_interface/EffortJointInterface</hardwareInterface>
-          <!-- <hardwareInterface>hardware_interface/PositionJointInterface</hardwareInterface> -->
       </joint>
   </transmission>

File: hand_simulator/urdf/hand_T42.xacro (robot description, xacro)
@@ -107,10 +107,10 @@
             </geometry>
         </visual>
-        <!-- <collision>
-            <origin xyz="0.000000 0.000000 -0.031750" />
-            <geometry>
-                <box size="0.038100 0.019050 0.078740" />
-            </geometry>
-        </collision> -->
+        <collision>
+            <origin xyz="-0.015875 -0.009000 -0.071550" />
+            <geometry>
+                <mesh filename="package://hand_simulator/meshes/proximal_t42.STL" scale="0.025400 0.025400 0.025400" />
+            </geometry>
+        </collision>
     </link>
     <gazebo reference="finger_1_1">
@@ -133,10 +133,10 @@
             </geometry>
         </visual>
-        <!-- <collision>
+        <collision>
             <origin xyz="-0.015875 -0.011709 -0.048006" />
             <geometry>
                 <mesh filename="package://hand_simulator/meshes/distal_t42.STL" scale="0.025400 0.025400 0.025400" />
             </geometry>
-        </collision> -->
+        </collision>
     </link>
     <gazebo reference="finger_1_2">
@@ -177,10 +177,10 @@
             </geometry>
         </visual>
-        <!-- <collision>
-            <origin xyz="0.000000 0.000000 -0.031750" />
-            <geometry>
-                <box size="0.038100 0.019050 0.078740" />
-            </geometry>
-        </collision> -->
+        <collision>
+            <origin xyz="-0.015875 -0.009000 -0.071550" />
+            <geometry>
+                <mesh filename="package://hand_simulator/meshes/proximal_t42.STL" scale="0.025400 0.025400 0.025400" />
+            </geometry>
+        </collision>
     </link>
     <gazebo reference="finger_2_1">
@@ -203,10 +203,10 @@
             </geometry>
         </visual>
-        <!-- <collision>
+        <collision>
             <origin xyz="-0.015875 -0.011709 -0.048006" />
             <geometry>
                 <mesh filename="package://hand_simulator/meshes/distal_t42.STL" scale="0.025400 0.025400 0.025400" />
             </geometry>
-        </collision> -->
+        </collision>
     </link>
     <gazebo reference="finger_2_2">
@@ -223,13 +223,13 @@
         <child link="rail"/>
         <origin
-          xyz="0.37 0 0.25"
+          xyz="0.37 0 0.4"
           rpy="0 0 0" />
     </joint>
     <joint name="rail_to_base" type="prismatic">
-        <origin rpy="0 0 0" xyz="0 0.000000 0." />
+        <origin rpy="0 0 0" xyz="-0.06 0.000000 0.2" />
         <parent link="rail" />
         <child link="base_link" />
-        <axis xyz="0 1 0"/>
-        <limit effort="1000.0" lower="-100." upper="100." velocity="4"/>
+        <axis xyz="0 0 1"/>
+        <limit effort="1000.0" lower="-100." upper="100." velocity="1"/>
     </joint>
     <joint name="base_link_to_swivel_1" type="fixed">
@@ -244,5 +244,5 @@
         <limit effort="10000" lower="0.0" upper="3.0" velocity="2" />
         <axis xyz="1 0 0" />
-        <dynamics damping="0" friction="0.0" />
+        <dynamics damping="5" friction="0.0" />
     </joint>
     <joint name="finger_1_1_to_finger_1_2" type="revolute">
@@ -252,5 +252,5 @@
         <limit effort="10000" lower="0.0" upper="1.57" velocity="2" />
         <axis xyz="1 0 0" />
-        <dynamics damping="0" friction="0.0" />
+        <dynamics damping="5" friction="0.0" />
     </joint>
     <joint name="base_link_to_swivel_2" type="fixed">
@@ -265,5 +265,5 @@
         <limit effort="10000" lower="0.0" upper="3.0" velocity="2" />
         <axis xyz="1 0 0" />
-        <dynamics damping="0" friction="0.0" />
+        <dynamics damping="5" friction="0.0" />
     </joint>
     <joint name="finger_2_1_to_finger_2_2" type="revolute">
@@ -271,7 +271,7 @@
         <parent link="finger_2_1" />
         <child link="finger_2_2" />
-        <limit effort="10000" lower="0.0" upper="3.0" velocity="2" />
+        <limit effort="10000" lower="0.0" upper="1.57" velocity="2" />
         <axis xyz="1 0 0" />
-        <dynamics damping="0" friction="0.0" />
+        <dynamics damping="5" friction="0.0" />
     </joint>
  <!-- Transmissions -->
@@ -291,6 +291,5 @@
       </actuator>
       <joint name="base_to_finger_1_1">
-          <!-- <hardwareInterface>hardware_interface/EffortJointInterface</hardwareInterface> -->
-          <hardwareInterface>hardware_interface/PositionJointInterface</hardwareInterface>
+          <hardwareInterface>hardware_interface/EffortJointInterface</hardwareInterface>
       </joint>
   </transmission>
@@ -301,6 +300,5 @@
       </actuator>
       <joint name="finger_1_1_to_finger_1_2">
-          <!-- <hardwareInterface>hardware_interface/EffortJointInterface</hardwareInterface> -->
-          <hardwareInterface>hardware_interface/PositionJointInterface</hardwareInterface>
+          <hardwareInterface>hardware_interface/EffortJointInterface</hardwareInterface>
       </joint>
   </transmission>
@@ -311,6 +309,5 @@
       </actuator>
       <joint name="base_to_finger_2_1">
-          <!-- <hardwareInterface>hardware_interface/EffortJointInterface</hardwareInterface> -->
-          <hardwareInterface>hardware_interface/PositionJointInterface</hardwareInterface>
+          <hardwareInterface>hardware_interface/EffortJointInterface</hardwareInterface>
       </joint>
   </transmission>
@@ -321,6 +318,5 @@
       </actuator>
       <joint name="finger_2_1_to_finger_2_2">
-          <!-- <hardwareInterface>hardware_interface/EffortJointInterface</hardwareInterface> -->
-          <hardwareInterface>hardware_interface/PositionJointInterface</hardwareInterface>
+          <hardwareInterface>hardware_interface/EffortJointInterface</hardwareInterface>
       </joint>
   </transmission>

File: hand_simulator/urdf/hand_reflex.xacro (robot description, xacro)
@@ -374,5 +374,5 @@
       <parent link="base_link"/>
       <child link="finger_1_1"/>
-      <limit effort="1000.0" lower="0." upper="1.57" velocity="0.5"/>
+      <limit effort="1000.0" lower="0." upper="1.57" velocity="200"/>
       <axis xyz="0 0 -1"/>
       <origin
@@ -403,5 +403,5 @@
       <parent link="base_link"/>
       <child link="finger_2_1"/>
-      <limit effort="1000.0" lower="-1.57" upper="0." velocity="0.5"/>
+      <limit effort="1000.0" lower="-1.57" upper="0." velocity="200"/>
       <axis xyz="0 0 -1"/>
       <origin
@@ -480,5 +480,4 @@
       <joint name="finger_1_1_to_finger_1_2">
           <hardwareInterface>hardware_interface/EffortJointInterface</hardwareInterface>
-      </joint>
   </transmission>
   <transmission name="finger1_3_trans" type="SimpleTransmission">
@@ -489,5 +488,4 @@
       <joint name="finger_1_2_to_finger_1_3">
           <hardwareInterface>hardware_interface/EffortJointInterface</hardwareInterface>
-      </joint>
   </transmission>
   <transmission name="finger2_1_trans" type="SimpleTransmission">
@@ -507,5 +505,4 @@
       <joint name="finger_2_1_to_finger_2_2">
           <hardwareInterface>hardware_interface/EffortJointInterface</hardwareInterface>
-      </joint>
   </transmission>
   <transmission name="finger2_3_trans" type="SimpleTransmission">
@@ -516,5 +513,4 @@
       <joint name="finger_2_2_to_finger_2_3">
           <hardwareInterface>hardware_interface/EffortJointInterface</hardwareInterface>
-      </joint>
   </transmission>
   <transmission name="finger2_3_trans" type="SimpleTransmission">
@@ -525,5 +521,4 @@
       <joint name="base_to_finger_3_2">
           <hardwareInterface>hardware_interface/EffortJointInterface</hardwareInterface>
-      </joint>
   </transmission>
   <transmission name="finger3_3_trans" type="SimpleTransmission">
