Commit message: T42 urdf and controller

File: hand_simulator/urdf/hand_T42.xacro (robot description, xacro)
@@ -92,5 +92,5 @@
       <material>Gazebo/Red</material>
     </gazebo>
-    <link name="finger_1_2">
+    <link name="finger_1_1">
         <inertial>
             <origin xyz="-0.015875 -0.009000 -0.071550" />
@@ -114,9 +114,9 @@
         </collision> -->
     </link>
-    <gazebo reference="finger_1_2">
-      <selfCollide>ture</selfCollide>
-      <material>Gazebo/Red</material>
-    </gazebo>
-    <link name="finger_1_3">
+    <gazebo reference="finger_1_1">
+      <selfCollide>true</selfCollide>
+      <material>Gazebo/Red</material>
+    </gazebo>
+    <link name="finger_1_2">
         <inertial>
             <origin xyz="-0.015875 -0.011709 -0.048006" />
@@ -140,5 +140,5 @@
         </collision> -->
     </link>
-    <gazebo reference="finger_1_3">
+    <gazebo reference="finger_1_2">
       <selfCollide>true</selfCollide>
       <mu1>${rubber_friction_coefficient}</mu1>
@@ -162,5 +162,5 @@
       <material>Gazebo/Red</material>
     </gazebo>
-    <link name="finger_2_2">
+    <link name="finger_2_1">
         <inertial>
             <origin xyz="-0.015875 -0.009000 -0.071550" />
@@ -184,9 +184,9 @@
         </collision> -->
     </link>
-    <gazebo reference="finger_2_2">
-      <selfCollide>true</selfCollide>
-      <material>Gazebo/Red</material>
-    </gazebo>
-    <link name="finger_2_3">
+    <gazebo reference="finger_2_1">
+      <selfCollide>true</selfCollide>
+      <material>Gazebo/Red</material>
+    </gazebo>
+    <link name="finger_2_2">
         <inertial>
             <origin xyz="-0.015875 -0.011709 -0.048006" />
@@ -210,5 +210,5 @@
         </collision> -->
     </link>
-    <gazebo reference="finger_2_3">
+    <gazebo reference="finger_2_2">
       <selfCollide>true</selfCollide>
       <mu1>${rubber_friction_coefficient}</mu1>
@@ -238,17 +238,17 @@
         <child link="swivel_1" />
     </joint>
-    <joint name="base_to_finger_1_2" type="revolute">
+    <joint name="base_to_finger_1_1" type="revolute">
         <origin rpy="1.57079632679 -1.57079632679 0" xyz="-0.016510 ${swivel_distance} 0.0000" />
         <parent link="base_link" />
-        <child link="finger_1_2" />
+        <child link="finger_1_1" />
         <limit effort="10000" lower="0.0" upper="3.0" velocity="2" />
         <axis xyz="1 0 0" />
         <dynamics damping="0" friction="0.0" />
     </joint>
-    <joint name="finger_1_2_to_finger_1_3" type="revolute">
+    <joint name="finger_1_1_to_finger_1_2" type="revolute">
         <origin rpy="0 0 0" xyz="0.000000 0.000000 -0.062551" />
-        <parent link="finger_1_2" />
-        <child link="finger_1_3" />
-        <limit effort="10000" lower="0.0" upper="3.0" velocity="2" />
+        <parent link="finger_1_1" />
+        <child link="finger_1_2" />
+        <limit effort="10000" lower="0.0" upper="1.57" velocity="2" />
         <axis xyz="1 0 0" />
         <dynamics damping="0" friction="0.0" />
@@ -259,7 +259,15 @@
         <child link="swivel_2" />
     </joint>
-    <joint name="base_to_finger_2_2" type="revolute">
+    <joint name="base_to_finger_2_1" type="revolute">
         <origin rpy="-1.57079632679 1.57079632679 0" xyz="-0.016510 -${swivel_distance} 0.000000" />
         <parent link="base_link" />
+        <child link="finger_2_1" />
+        <limit effort="10000" lower="0.0" upper="3.0" velocity="2" />
+        <axis xyz="1 0 0" />
+        <dynamics damping="0" friction="0.0" />
+    </joint>
+    <joint name="finger_2_1_to_finger_2_2" type="revolute">
+        <origin rpy="0 0 0" xyz="0.000000 0.000000 -0.062551" />
+        <parent link="finger_2_1" />
         <child link="finger_2_2" />
         <limit effort="10000" lower="0.0" upper="3.0" velocity="2" />
@@ -267,12 +275,4 @@
         <dynamics damping="0" friction="0.0" />
     </joint>
-    <joint name="prox_to_finger_2_3" type="revolute">
-        <origin rpy="0 0 0" xyz="0.000000 0.000000 -0.062551" />
-        <parent link="finger_2_2" />
-        <child link="finger_2_3" />
-        <limit effort="10000" lower="0.0" upper="3.0" velocity="2" />
-        <axis xyz="1 0 0" />
-        <dynamics damping="0" friction="0.0" />
-    </joint>
  <!-- Transmissions -->
   <transmission name="lift" type="SimpleTransmission">
@@ -290,6 +290,7 @@
           <mechanicalReduction>1</mechanicalReduction>
       </actuator>
-      <joint name="base_to_finger_1_2">
-          <hardwareInterface>hardware_interface/EffortJointInterface</hardwareInterface>
+      <joint name="base_to_finger_1_1">
+          <!-- <hardwareInterface>hardware_interface/EffortJointInterface</hardwareInterface> -->
+          <hardwareInterface>hardware_interface/PositionJointInterface</hardwareInterface>
       </joint>
   </transmission>
@@ -299,6 +300,7 @@
           <mechanicalReduction>1</mechanicalReduction>
       </actuator>
-      <joint name="finger_1_2_to_finger_1_3">
-          <hardwareInterface>hardware_interface/EffortJointInterface</hardwareInterface>
+      <joint name="finger_1_1_to_finger_1_2">
+          <!-- <hardwareInterface>hardware_interface/EffortJointInterface</hardwareInterface> -->
+          <hardwareInterface>hardware_interface/PositionJointInterface</hardwareInterface>
       </joint>
   </transmission>
@@ -308,6 +310,7 @@
           <mechanicalReduction>1</mechanicalReduction>
       </actuator>
-      <joint name="base_to_finger_2_2">
-          <hardwareInterface>hardware_interface/EffortJointInterface</hardwareInterface>
+      <joint name="base_to_finger_2_1">
+          <!-- <hardwareInterface>hardware_interface/EffortJointInterface</hardwareInterface> -->
+          <hardwareInterface>hardware_interface/PositionJointInterface</hardwareInterface>
       </joint>
   </transmission>
@@ -317,6 +320,7 @@
           <mechanicalReduction>1</mechanicalReduction>
       </actuator>
-      <joint name="finger_2_2_to_finger_2_3">
-          <hardwareInterface>hardware_interface/EffortJointInterface</hardwareInterface>
+      <joint name="finger_2_1_to_finger_2_2">
+          <!-- <hardwareInterface>hardware_interface/EffortJointInterface</hardwareInterface> -->
+          <hardwareInterface>hardware_interface/PositionJointInterface</hardwareInterface>
       </joint>
   </transmission>

Commit message: Finalized the hand models

File: hand_simulator/urdf/hand_T42.xacro (robot description, xacro)
@@ -83,5 +83,5 @@
                 <color rgba="1.0 1.0 1.0 1.0" />
             </material>
-            <origin rpy="0 1.57 1.57" xyz="-0.016510 -${swivel_distance} 0" />
+            <origin rpy="0 1.57 1.57" xyz="-0.016510 ${swivel_distance} 0" />
             <geometry>
                 <mesh filename="package://hand_simulator/meshes/swivel_t42.STL" scale="0.001 0.001 0.001" />
@@ -125,6 +125,6 @@
         </inertial>
         <visual>
-            <material name="orange">
-                <color rgba="0.9 0.3 0.1 1.0" />
+            <material name="green">
+                <color rgba="0.1 1.0 0.1 1.0" />
             </material>
             <origin xyz="-0.015875 -0.011709 -0.048006" />
@@ -153,5 +153,5 @@
                 <color rgba="1.0 1.0 1.0 1.0" />
             </material>
-            <origin rpy="0 1.57 1.57" xyz="-0.016510 ${swivel_distance} 0" />
+            <origin rpy="0 1.57 1.57" xyz="-0.016510 -${swivel_distance} 0" />
             <geometry>
                 <mesh filename="package://hand_simulator/meshes/swivel_t42.STL" scale="0.001 0.001 0.001" />
@@ -195,6 +195,6 @@
         </inertial>
         <visual>
-            <material name="green">
-                <color rgba="0.1 1.0 0.1 1.0" />
+            <material name="orange">
+                <color rgba="0.9 0.3 0.1 1.0" />
             </material>
             <origin xyz="-0.015875 -0.011709 -0.048006" />
@@ -218,11 +218,71 @@
       <material>Gazebo/Red</material>
     </gazebo>
+    <!-- Camera -->
+    <xacro:property name="camera_size" value="0.1" /> <!-- Size of square 'camera' box -->
+    <link name="camera_link">
+        <visual>
+            <origin xyz="0 0 0" rpy="0 0 0"/>
+            <geometry>
+                <box size="${camera_size} ${camera_size} ${camera_size}"/>
+            </geometry>
+            <material name="black"/>
+        </visual>
+    </link>
+    <gazebo reference="camera_link">
+        <material>Gazebo/Black</material>
+        <sensor type="camera" name="camera">
+            <update_rate>30.0</update_rate>
+            <camera name="head">
+                <horizontal_fov>1.3962634</horizontal_fov>
+                <image>
+                <width>800</width>
+                <height>800</height>
+                <format>R8G8B8</format>
+                </image>
+                <clip>
+                <near>0.02</near>
+                <far>300</far>
+                </clip>
+                <noise>
+                <type>gaussian</type>
+                <!-- Noise is sampled independently per pixel on each frame.
+                    That pixel's noise value is added to each of its color
+                    channels, which at that point lie in the range [0,1]. -->
+                <mean>0.0</mean>
+                <stddev>0.007</stddev>
+                </noise>
+            </camera>
+            <plugin name="camera_controller" filename="libgazebo_ros_camera.so">
+                <alwaysOn>true</alwaysOn>
+                <updateRate>0.0</updateRate>
+                <cameraName>hand/camera</cameraName>
+                <imageTopicName>image_raw</imageTopicName>
+                <cameraInfoTopicName>camera_info</cameraInfoTopicName>
+                <frameName>camera_link</frameName>
+                <hackBaseline>0.07</hackBaseline>
+                <distortionK1>0.0</distortionK1>
+                <distortionK2>0.0</distortionK2>
+                <distortionK3>0.0</distortionK3>
+                <distortionT1>0.0</distortionT1>
+                <distortionT2>0.0</distortionT2>
+            </plugin>
+        </sensor>
+    </gazebo>
   <!-- Joints -->
     <joint name="world_to_rail" type="fixed">
         <parent link="world"/>
         <child link="rail"/>
+      <selfCollide>false</selfCollide>
         <origin
           xyz="0.37 0 0.4"
           rpy="0 0 0" />
+    </joint>
+    <joint name="rail_to_camera" type="fixed">
+        <parent link="rail"/>
+        <child link="camera_link"/>
+        <axis xyz="0 0 -1" />
+        <origin
+          xyz="-0.2 0 0.7"
+          rpy="0 1.57 3.14" />
     </joint>
     <joint name="rail_to_base" type="prismatic">
@@ -239,5 +299,5 @@
     </joint>
     <joint name="base_to_finger_1_1" type="revolute">
-        <origin rpy="1.57079632679 -1.57079632679 0" xyz="-0.016510 ${swivel_distance} 0.0000" />
+        <origin rpy="-1.57079632679 1.57079632679 0" xyz="-0.016510 -${swivel_distance} 0.000000" />
         <parent link="base_link" />
         <child link="finger_1_1" />
@@ -260,5 +320,5 @@
     </joint>
     <joint name="base_to_finger_2_1" type="revolute">
-        <origin rpy="-1.57079632679 1.57079632679 0" xyz="-0.016510 -${swivel_distance} 0.000000" />
+        <origin rpy="1.57079632679 -1.57079632679 0" xyz="-0.016510 ${swivel_distance} 0.0000" />
         <parent link="base_link" />
         <child link="finger_2_1" />
